File: placas/EduRoMAA-EduCIAA/EduRoMAA-EduCIAA.kicad_pcb (KiCad board)
At the start: 2 copper layers, 103 x 80 mm, 81 parts, among them J1 DC_IN, J2 Motor_Izq, J3 Motor_Der, J4 Bluetooth, J5 Sonar, J6 DC_OUT, J7 DC_IN, Q1 BC548, Q2 BC548, Q3 BC548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

Commit message: Agrego BOM, PDF y modifico esquematico
Se modifica las resistencias R5,R6 a 3,3kohm. Se modifica fp
de uno de los TCRT5000, agrego pdf de serigrafia frontal,
pistas inferiores y archivos para fabricacion.
Agrego BOM, interactivo y html.
Parts:
- R5, R6: value 10k -> 3.3k
Routing:
- net GND_IRLED1: track 17.5 -> 18.4 mm
